File: test2/test2.kicad_sch (KiCad schematic)
At the start: 0 parts

Commit message: Changed title to c1
Other:
- company: (none) -> AutoIntern2
- title: (none) -> Sheet2
Changed lines of the file:
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@@
 	(generator_version "10.0")
 	(paper "A4")
+	(title_block
+		(title "Sheet2")
+		(date "2026-07-01")
+		(rev "v1.1.0")
+		(company "AutoIntern2")
+		(comment 1 "c1")
+	)
 	(sheet_instances
 		(path "/"
